File: board/hall.sch (KiCad schematic (older format))
At the start: 74 parts, among them U1 74HC238, U10 A3144, U11 A3144, U12 A3144, U13 A3144, U14 A3144, U15 A3144, U16 A3144, U17 A3144, U18 A3144, U19 A3144, U2 74LS151, U20 A3144, U21 A3144, U22 A3144, U23 A3144, U24 A3144, U25 A3144, U26 A3144, U27 A3144, U28 A3144, U29 A3144, U3 A3144, U30 A3144, U31 A3144, U32 A3144, U33 A3144, U34 A3144, U35 A3144, U36 A3144, U37 A3144, U38 A3144, U39 A3144, U4 A3144, U40 A3144, U41 A3144, U42 A3144, U43 A3144, U44 A3144, U45 A3144, U46 A3144, U47 A3144, U48 A3144, U49 A3144, U5 A3144, U50 A3144, U51 A3144, U52 A3144, U53 A3144, U54 A3144, U55 A3144, U56 A3144, U57 A3144, U58 A3144, U59 A3144, U6 A3144, U60 A3144, U61 A3144, U62 A3144, U63 A3144, U64 A3144, U65 A3144, U66 A3144, U7 A3144, U8 A3144, U9 A3144

Commit message: Folder reorganized: board
Parts:
- U10, U11, U12, U13, U14, U15, U16, U17, U18, U19, U20, U21, U22, U23, U24, U25, U26, U27, U28, U29, U3, U30, U31, U32, U33, U34, U35, U36, U37, U38, U39, U4, U40, U41, U42, U43, U44, U45, U46, U47, U48, U49, U5, U50, U51, U52, U53, U54, U55, U56, U57, U58, U59, U6, U60, U61, U62, U63, U64, U65, U66, U7, U8, U9: symbol board:A3144 -> Board:A3144
Changed lines of the file:
@@
 	6450 3450 6025 3450
 $Comp
-L board:A3144 U4
+L Board:A3144 U4
 U 1 1 60369E87
 P 6550 3475
@@
 	7725 3450 7300 3450
 $Comp
-L board:A3144 U12
+L Board:A3144 U12
 U 1 1 604A0EC4
 P 7825 3475
@@
 	9000 3450 8575 3450
 $Comp
-L board:A3144 U20
+L Board:A3144 U20
 U 1 1 6052829F
 P 9100 3475
@@
 	10275 3450 9850 3450
 $Comp
-L board:A3144 U28
+L Board:A3144 U28
 U 1 1 6052837F
 P 10375 3475
@@
 	11550 3450 11125 3450
 $Comp
-L board:A3144 U36
+L Board:A3144 U36
 U 1 1 6054B91A
 P 11650 3475
@@
 	12825 3450 12400 3450
 $Comp
-L board:A3144 U44
+L Board:A3144 U44
 U 1 1 6054B9FA
 P 12925 3475
@@
 	14100 3450 13675 3450
 $Comp
-L board:A3144 U52
+L Board:A3144 U52
 U 1 1 60582E07
 P 14200 3475
@@
 	15375 3450 14950 3450
 $Comp
-L board:A3144 U60
+L Board:A3144 U60
 U 1 1 60582EE7
 P 15475 3475
@@
 Connection ~ 15800 11625
 $Comp
-L board:A3144 U11
+L Board:A3144 U11
 U 1 1 5FDB7CA5
 P 7825 2200
@@
 $EndComp
 $Comp
-L board:A3144 U19
+L Board:A3144 U19
 U 1 1 5FDB848C
 P 9100 2200
@@
 $EndComp
 $Comp
-L board:A3144 U27
+L Board:A3144 U27
 U 1 1 5FDB898D
 P 10375 2200
@@
 $EndComp
 $Comp
-L board:A3144 U35
+L Board:A3144 U35
 U 1 1 5FDB8E73
 P 11650 2200
@@
 $EndComp
 $Comp
-L board:A3144 U43
+L Board:A3144 U43
 U 1 1 5FDB96CF
 P 12925 2200
@@
 $EndComp
 $Comp
-L board:A3144 U51
+L Board:A3144 U51
 U 1 1 5FDB9C5B
 P 14200 2200
@@
 $EndComp
 $Comp
-L board:A3144 U59
+L Board:A3144 U59
 U 1 1 5FDBA153
 P 15475 2200
@@
 $EndComp
 $Comp
-L board:A3144 U13
+L Board:A3144 U13
 U 1 1 60E3C5AB
 P 7825 4750
@@
 $EndComp
 $Comp
-L board:A3144 U21
+L Board:A3144 U21
 U 1 1 60E3C5B1
 P 9100 4750
@@
 $EndComp
 $Comp
-L board:A3144 U29
+L Board:A3144 U29
 U 1 1 60E3C5B7
 P 10375 4750
@@
 $EndComp
 $Comp
-L board:A3144 U37
+L Board:A3144 U37
 U 1 1 60E3C5BD
 P 11650 4750
@@
 $EndComp
 $Comp
-L board:A3144 U45
+L Board:A3144 U45
 U 1 1 60E3C5C3
 P 12925 4750
@@
 $EndComp
 $Comp
-L board:A3144 U53
+L Board:A3144 U53
 U 1 1 60E3C5C9
 P 14200 4750
@@
 $EndComp
 $Comp
-L board:A3144 U5
+L Board:A3144 U5
 U 1 1 60E3C5CF
 P 6550 4750
@@
 $EndComp
 $Comp
-L board:A3144 U61
+L Board:A3144 U61
 U 1 1 60E3C5D5
 P 15475 4750
@@
 $EndComp
 $Comp
-L board:A3144 U14
+L Board:A3144 U14
 U 1 1 60EA060B
 P 7825 6025
@@
 $EndComp
 $Comp
-L board:A3144 U22
+L Board:A3144 U22
 U 1 1 60EA0611
 P 9100 6025
@@
 $EndComp
 $Comp
-L board:A3144 U30
+L Board:A3144 U30
 U 1 1 60EA0617
 P 10375 6025
@@
 $EndComp
 $Comp
-L board:A3144 U38
+L Board:A3144 U38
 U 1 1 60EA061D
 P 11650 6025
@@
 $EndComp
 $Comp
-L board:A3144 U46
+L Board:A3144 U46
 U 1 1 60EA0623
 P 12925 6025
@@
 $EndComp
 $Comp
-L board:A3144 U54
+L Board:A3144 U54
 U 1 1 60EA0629
 P 14200 6025
@@
 $EndComp
 $Comp
-L board:A3144 U6
+L Board:A3144 U6
 U 1 1 60EA062F
 P 6550 6025
@@
 $EndComp
 $Comp
-L board:A3144 U62
+L Board:A3144 U62
 U 1 1 60EA0635
 P 15475 6025
@@
 $EndComp
 $Comp
-L board:A3144 U15
+L Board:A3144 U15
 U 1 1 60F04401
 P 7825 7300
@@
 $EndComp
 $Comp
-L board:A3144 U23
+L Board:A3144 U23
 U 1 1 60F04407
 P 9100 7300
@@
 $EndComp
 $Comp
-L board:A3144 U31
+L Board:A3144 U31
 U 1 1 60F0440D
 P 10375 7300
@@
 $EndComp
 $Comp
-L board:A3144 U39
+L Board:A3144 U39
 U 1 1 60F04413
 P 11650 7300
@@
 $EndComp
 $Comp
-L board:A3144 U47
+L Board:A3144 U47
 U 1 1 60F04419
 P 12925 7300
@@
 $EndComp
 $Comp
-L board:A3144 U55
+L Board:A3144 U55
 U 1 1 60F0441F
 P 14200 7300
@@
 $EndComp
 $Comp
-L board:A3144 U7
+L Board:A3144 U7
 U 1 1 60F04425
 P 6550 7300
@@
 $EndComp
 $Comp
-L board:A3144 U63
+L Board:A3144 U63
 U 1 1 60F0442B
 P 15475 7300
@@
 $EndComp
 $Comp
-L board:A3144 U16
+L Board:A3144 U16
 U 1 1 60F6874B
 P 7825 8575
@@
 $EndComp
 $Comp
-L board:A3144 U32
+L Board:A3144 U32
 U 1 1 60F68757
 P 10375 8575
@@
 $EndComp
 $Comp
-L board:A3144 U40
+L Board:A3144 U40
 U 1 1 60F6875D
 P 11650 8575
@@
 $EndComp
 $Comp
-L board:A3144 U48
+L Board:A3144 U48
 U 1 1 60F68763
 P 12925 8575
@@
 $EndComp
 $Comp
-L board:A3144 U56
+L Board:A3144 U56
 U 1 1 60F68769
 P 14200 8575
@@
 $EndComp
 $Comp
-L board:A3144 U8
+L Board:A3144 U8
 U 1 1 60F6876F
 P 6550 8575
@@
 $EndComp
 $Comp
-L board:A3144 U64
+L Board:A3144 U64
 U 1 1 60F68775
 P 15475 8575
@@
 $EndComp
 $Comp
-L board:A3144 U17
+L Board:A3144 U17
 U 1 1 60FCD807
 P 7825 9850
@@
 $EndComp
 $Comp
-L board:A3144 U25
+L Board:A3144 U25
 U 1 1 60FCD80D
 P 9100 9850
@@
 $EndComp
 $Comp
-L board:A3144 U33
+L Board:A3144 U33
 U 1 1 60FCD813
 P 10375 9850
@@
 $EndComp
 $Comp
-L board:A3144 U41
+L Board:A3144 U41
 U 1 1 60FCD819
 P 11650 9850
@@
 $EndComp
 $Comp
-L board:A3144 U49
+L Board:A3144 U49
 U 1 1 60FCD81F
 P 12925 9850
@@
 $EndComp
 $Comp
-L board:A3144 U57
+L Board:A3144 U57
 U 1 1 60FCD825
 P 14200 9850
@@
 $EndComp
 $Comp
-L board:A3144 U9
+L Board:A3144 U9
 U 1 1 60FCD82B
 P 6550 9850
@@
 $EndComp
 $Comp
-L board:A3144 U65
+L Board:A3144 U65
 U 1 1 60FCD831
 P 15475 9850
@@
 $EndComp
 $Comp
-L board:A3144 U18
+L Board:A3144 U18
 U 1 1 61031773
 P 7825 11125
@@
 $EndComp
 $Comp
-L board:A3144 U26
+L Board:A3144 U26
 U 1 1 61031779
 P 9100 11125
@@
 $EndComp
 $Comp
-L board:A3144 U34
+L Board:A3144 U34
 U 1 1 6103177F
 P 10375 11125
@@
 $EndComp
 $Comp
-L board:A3144 U50
+L Board:A3144 U50
 U 1 1 6103178B
 P 12925 11125
@@
 $EndComp
 $Comp
-L board:A3144 U58
+L Board:A3144 U58
 U 1 1 61031791
 P 14200 11125
@@
 $EndComp
 $Comp
-L board:A3144 U66
+L Board:A3144 U66
 U 1 1 6103179D
 P 15475 11125
@@
 $EndComp
 $Comp
-L board:A3144 U3
+L Board:A3144 U3
 U 1 1 5FDB5685
 P 6550 2200
@@
 $EndComp
 $Comp
-L board:A3144 U24
+L Board:A3144 U24
 U 1 1 60F68751
 P 9100 8575
@@
 $EndComp
 $Comp
-L board:A3144 U10
+L Board:A3144 U10
 U 1 1 61031797
 P 6550 11125
@@
 $EndComp
 $Comp
-L board:A3144 U42
+L Board:A3144 U42
 U 1 1 61031785
 P 11650 11125
